Commit message: urdf 模型场景

File: src/scene_generation/object/contactdb/airplane/airplane.urdf (robot description, URDF)
Before this commit: robot object, 1 links, 0 joints
Links:
- link object: mass None -> 0.100000

File: src/scene_generation/object/contactdb/alarm_clock/alarm_clock.urdf (robot description, URDF)
Before this commit: robot object, 1 links, 0 joints
Links:
- link object: mass None -> 0.100000

File: src/scene_generation/object/contactdb/apple/apple.urdf (robot description, URDF)
Before this commit: robot object, 1 links, 0 joints
Links:
- link object: mass None -> 0.100000

File: src/scene_generation/object/contactdb/banana/banana.urdf (robot description, URDF)
Before this commit: robot object, 1 links, 0 joints
Links:
- link object: mass None -> 0.100000

File: src/scene_generation/object/contactdb/binoculars/binoculars.urdf (robot description, URDF)
Before this commit: robot object, 1 links, 0 joints
Links:
- link object: mass None -> 0.100000

File: src/scene_generation/object/contactdb/bowl/bowl.urdf (robot description, URDF)
Before this commit: robot object, 1 links, 0 joints
Links:
- link object: mass None -> 0.100000

File: src/scene_generation/object/contactdb/camera/camera.urdf (robot description, URDF)
Before this commit: robot object, 1 links, 0 joints
Links:
- link object: mass None -> 0.100000

File: src/scene_generation/object/contactdb/cell_phone/cell_phone.urdf (robot description, URDF)
Before this commit: robot object, 1 links, 0 joints
Links:
- link object: mass None -> 0.100000

File: src/scene_generation/object/contactdb/cube_large/cube_large.urdf (robot description, URDF)
Before this commit: robot object, 1 links, 0 joints
Links:
- link object: mass None -> 0.100000

File: src/scene_generation/object/contactdb/cube_medium/cube_medium.urdf (robot description, URDF)
Before this commit: robot object, 1 links, 0 joints
Links:
- link object: mass None -> 0.100000

File: src/scene_generation/object/contactdb/cube_small/cube_small.urdf (robot description, URDF)
Before this commit: robot object, 1 links, 0 joints
Links:
- link object: mass None -> 0.100000

File: src/scene_generation/object/contactdb/cup/cup.urdf (robot description, URDF)
Before this commit: robot object, 1 links, 0 joints
Links:
- link object: mass None -> 0.100000

File: src/scene_generation/object/contactdb/cylinder_large/cylinder_large.urdf (robot description, URDF)
Before this commit: robot object, 1 links, 0 joints
Links:
- link object: mass None -> 0.100000

File: src/scene_generation/object/contactdb/cylinder_medium/cylinder_medium.urdf (robot description, URDF)
Before this commit: robot object, 1 links, 0 joints
Links:
- link object: mass None -> 0.100000

File: src/scene_generation/object/contactdb/cylinder_small/cylinder_small.urdf (robot description, URDF)
Before this commit: robot object, 1 links, 0 joints
Links:
- link object: mass None -> 0.100000

File: src/scene_generation/object/contactdb/door_knob/door_knob.urdf (robot description, URDF)
Before this commit: robot object, 1 links, 0 joints
Links:
- link object: mass None -> 0.100000

File: src/scene_generation/object/contactdb/elephant/elephant.urdf (robot description, URDF)
Before this commit: robot object, 1 links, 0 joints
Links:
- link object: mass None -> 0.100000

File: src/scene_generation/object/contactdb/eyeglasses/eyeglasses.urdf (robot description, URDF)
Before this commit: robot object, 1 links, 0 joints
Links:
- link object: mass None -> 0.100000

File: src/scene_generation/object/contactdb/flashlight/flashlight.urdf (robot description, URDF)
Before this commit: robot object, 1 links, 0 joints
Links:
- link object: mass None -> 0.100000

File: src/scene_generation/object/contactdb/flute/flute.urdf (robot description, URDF)
Before this commit: robot object, 1 links, 0 joints
Links:
- link object: mass None -> 0.100000
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